Commit message: Make base_joint a revolute joint

File: ros2_control_test_assets/urdf/test_description_mock.urdf (robot description, URDF)
Before this commit: robot MinimalRobot, 4 links, 3 joints
Joints:
- joint base_joint: limit (none) -> lower=-3.14159265359 upper=3.14159265359 effort=0.1 velocity=0.2; type fixed -> revolute
